File: Hardware/SparkFun_AirQuality_Combo.kicad_sch (KiCad schematic)
At the start: 35 parts, among them J1 Qwiic_RA, J2 Qwiic_RA, J3 Conn_01x04, U1 AP3012, U1 SEN55, U3 SCD41, U4 SEN55_Outline

Commit message: Pre design review changes
Parts:
- removed C1: 22uF, SparkFun-Capacitor:C_0603_1608Metric, symbol SparkFun-Capacitor:22uF_0603_6.3V_20%
- removed U7: ~, SparkFun-Aesthetic:Ordering_Instructions, symbol SparkFun-Aesthetic:Ordering_Instructions
- added C2: 22uF, SparkFun-Capacitor:C_0805_2012Metric, symbol SparkFun-Capacitor:22uF_0805_10V_20%
- JP1: value ~ -> PWR
- JP2: value ~ -> I2C
Connections:
- net 5V: now also C2.1
- net GND: now also C2.2
Other:
- note added: "Cut jumper to remove pullups from bus"
- note added: "Cut jumper to turn off power LED"
- note added: "Input Voltage: 2.7-5V"
- note added: "Max Current: 350mA"
- note added: "Vout=1.25*(1+R1/R2) R1=(Vout*0.8-1)*R2 R1 = 100k / R2 = 33k"
- title: (none) -> SparkFun Indoor Air Quality Sensor - SCD41 SEN55 (Qwiic)
- moved on the sheet: C1, C5, D1, L1, R2, R3, U1

Commit message: Pre design review updates
Parts:
- added C1: 0.1uF, SparkFun-Capacitor:C_0603_1608Metric, symbol SparkFun-Capacitor:0.1uF_0603_25V_20%
- C5: Tolerance +80%/-20% -> 20%
- JP1: value PWR -> ~
- JP2: value I2C -> ~
Connections:
- net 3.3V: now also C1.1
- net GND: now also C1.2
Changed lines of the file:
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@@
+    (stroke (width 0) (type default))
+  )
+  (wire (pts (xy 255.27 102.87) (xy 255.27 101.6))
     (stroke (width 0) (type default))
   )
@@
   )
   (wire (pts (xy 195.58 99.06) (xy 195.58 96.52))
+    (stroke (width 0) (type default))
+  )
+  (wire (pts (xy 255.27 92.71) (xy 255.27 93.98))
     (stroke (width 0) (type default))
   )
@@
     )
   )
+  (symbol (lib_id "SparkFun-Capacitor:0.1uF_0603_25V_20%") (at 255.27 97.79 0) (unit 1)
+    (in_bom yes) (on_board yes) (dnp no) (fields_autoplaced)
+    (property "Reference" "C1" (at 259.08 93.98 0)
+      (effects (font (size 1.27 1.27)) (justify left))
+    )
+    (property "Value" "0.1uF" (at 259.08 96.52 0)
+      (effects (font (size 1.27 1.27)) (justify left))
+    )
+    (property "Footprint" "SparkFun-Capacitor:C_0603_1608Metric" (at 255.27 109.22 0)
+      (effects (font (size 1.27 1.27)) hide)
+    )
+    (property "Datasheet" "https://cdn.sparkfun.com/assets/8/a/4/a/5/Kemet_Capacitor_Datasheet.pdf" (at 255.27 111.76 0)
+      (effects (font (size 1.27 1.27)) hide)
+    )
+    (property "PROD_ID" "CAP-00810" (at 255.27 114.3 0)
+      (effects (font (size 1.27 1.27)) hide)
+    )
+    (property "Voltage" "25V" (at 259.08 99.06 0)
+      (effects (font (size 1.27 1.27)) (justify left))
+    )
+    (property "Tolerance" "20%" (at 259.08 101.6 0)
+      (effects (font (size 1.27 1.27)) (justify left))
+    )
+    (pin "1")
+    (pin "2")
+    (instances
+      (project "SparkFun_AirQuality_Combo"
+        (path "/e3dd3ae4-244d-4cba-9cca-5d2abf83f29a"
+          (reference "C1") (unit 1)
+        )
+      )
+    )
+  )
   (symbol (lib_id "SparkFun-PowerSymbol:GND") (at 77.47 53.34 0) (unit 1)
     (in_bom yes) (on_board yes) (dnp no)
@@
       (effects (font (size 1.27 1.27)))
     )
-    (property "Value" "PWR" (at 57.15 110.49 0)
+    (property "Value" "~" (at 57.15 110.49 0)
       (effects (font (size 1.27 1.27)))
     )
@@
         (path "/e3dd3ae4-244d-4cba-9cca-5d2abf83f29a"
           (reference "R1") (unit 1)
+        )
+      )
+    )
+  )
+  (symbol (lib_id "SparkFun-PowerSymbol:3.3V") (at 255.27 92.71 0) (unit 1)
+    (in_bom yes) (on_board yes) (dnp no)
+    (property "Reference" "#PWR01" (at 255.27 96.52 0)
+      (effects (font (size 1.27 1.27)) hide)
+    )
+    (property "Value" "3.3V" (at 255.27 89.154 0)
+      (effects (font (size 1.27 1.27)))
+    )
+    (property "Footprint" "" (at 255.27 92.71 0)
+      (effects (font (size 1.27 1.27)) hide)
+    )
+    (property "Datasheet" "" (at 255.27 92.71 0)
+      (effects (font (size 1.27 1.27)) hide)
+    )
+    (pin "1")
+    (instances
+      (project "SparkFun_AirQuality_Combo"
+        (path "/e3dd3ae4-244d-4cba-9cca-5d2abf83f29a"
+          (reference "#PWR01") (unit 1)
         )
       )
@@
       (effects (font (size 1.27 1.27)) (justify left))
     )
-    (property "Tolerance" "+80%/-20%" (at 246.38 101.6 0)
+    (property "Tolerance" "20%" (at 246.38 101.6 0)
       (effects (font (size 1.27 1.27)) (justify left))
     )
@@
     )
   )
+  (symbol (lib_id "SparkFun-PowerSymbol:GND") (at 255.27 102.87 0) (unit 1)
+    (in_bom yes) (on_board yes) (dnp no)
+    (property "Reference" "#PWR02" (at 255.27 109.22 0)
+      (effects (font (size 1.27 1.27)) hide)
+    )
+    (property "Value" "GND" (at 255.27 106.68 0)
+      (effects (font (size 1.27 1.27)))
+    )
+    (property "Footprint" "" (at 255.27 102.87 0)
+      (effects (font (size 1.27 1.27)) hide)
+    )
+    (property "Datasheet" "" (at 255.27 102.87 0)
+      (effects (font (size 1.27 1.27)) hide)
+    )
+    (pin "1")
+    (instances
+      (project "SparkFun_AirQuality_Combo"
+        (path "/e3dd3ae4-244d-4cba-9cca-5d2abf83f29a"
+          (reference "#PWR02") (unit 1)
+        )
+      )
+    )
+  )
   (symbol (lib_id "SparkFun-PowerSymbol:3.3V") (at 229.87 92.71 0) (unit 1)
     (in_bom yes) (on_board yes) (dnp no)
@@
       (effects (font (size 1.27 1.27)))
     )
-    (property "Value" "I2C" (at 107.95 116.84 0)
-      (effects (font (size 1.27 1.27)))
-    )
+    (property "Value" "~" (at 107.95 116.84 0)
+      (effects (font (size 1.27 1.27)))
+    )

Commit message: Add PTH at 0.8"
Parts:
- added ST5: Standoff, SparkFun-Hardware:Standoff, symbol SparkFun-Hardware:Standoff
- added TP1: 0.75mm, SparkFun-Connector:TestPoint-0.75mm, symbol SparkFun-Connector:TestPoint_0.75mm
- added U2: ~, SparkFun-Aesthetic:Ordering_Instructions, symbol SparkFun-Aesthetic:Ordering_Instructions
Connections:
- net 5V: now also TP1.1
