File: Hardware/SparkFun Indoor Air Quality Sensor - SCD41 SEN55.kicad_pcb (KiCad board)
At the start: 2 copper layers, 82.5 x 44.5 mm, 59 parts, among them J1 Qwiic_RA, J2 Qwiic_RA, J3 Conn_01x04, U1 SEN55, U3 SCD41, U4 SEN55_Outline, U5 AP3012

Commit message: Fix PROD_ID on SEN55 connector and module.
Parts:
- removed U1: SEN55, SparkFun-Connector:JST_SMD_1.25mm-6_Locking
- removed U2: ~, SparkFun-Aesthetic:Ordering_Instructions
- added U6: SEN55_Connector, SparkFun-Connector:JST_SMD_1.25mm-6_Locking, F.Cu at (182.2, 109.9)

Commit message: Update 3D models
Parts:
- D1: footprint SparkFun-LED:LED_0603_1608Metric -> SparkFun-LED:LED_0603_1608Metric_Red
- U3: footprint SparkFun-Sensor:SCD4X -> SparkFun-Sensor:SCD4x
