File: Hardware/Production/SparkFun Indoor Air Quality Sensor - SCD41 SEN55_panelized.kicad_pcb (KiCad board)
At the start: 2 copper layers, 179.3 x 148 mm, 350 parts, among them J1 Qwiic_RA, J2 Qwiic_RA, J3 Conn_01x04, U1 SEN55, U3 SCD41, U4 SEN55_Outline, U5 AP3012

Commit message: File rename
Parts:
- removed the ? at (101.1, 121.2) (x2)
- removed the ? at (101.1, -9.16) (x2)
- removed the ? at (274.1, -9.16) (x2)
- added ?: , Fiducial_1.5mm_Mask3mm, F.Cu at (101.1, 121.2)
- added ?: , Fiducial_1mm_Mask3mm, F.Cu at (101.1, -9.16)
- added ?: , Fiducial_1mm_Mask3mm, F.Cu at (274.1, -9.16)
- added ?: , Fiducial_1.5mm_Mask3mm, B.Cu at (101.1, 121.2)
- added ?: , Fiducial_1mm_Mask3mm, B.Cu at (274.1, -9.16)
- added ?: , Fiducial_1mm_Mask3mm, B.Cu at (101.1, -9.16)
- moved G4 7.43 mm to (214.6, 175.3)
